Commit message: Add files via upload

File: manipulator/dummy_gazebo/robot/dummy.xacro (robot description, xacro)
@@ -1,7 +1,11 @@
 <?xml version='1.0' encoding='utf-8'?>
 <robot xmlns:xacro="http://www.ros.org/wiki/xacro" name="dummy">
+  <xacro:arg name="robot_name" default=""/>
+  <xacro:property name="namespace" value="$(arg robot_name)"/>
   <xacro:property name="description_package" value="dummy_description"/>
   <xacro:property name="gazebo_package" value="dummy_gazebo"/>
   <xacro:include filename="$(find ${description_package})/robot/dynamics/robot.xacro"/>
   <xacro:dummy_robot package="${description_package}"/>
+  <xacro:include filename="$(find ${gazebo_package})/robot/ros2_control.gazebo.xacro"/>
+  <xacro:controller_plugins namespace="${namespace}"/>
 </robot>

File: manipulator/dummy_gazebo/robot/ros2_control.gazebo.xacro (robot description, xacro)
@@ -1,3 +1,34 @@
 <?xml version='1.0' encoding='utf-8'?>
 <robot xmlns:xacro="http://www.ros.org/wiki/xacro">
+    <xacro:macro name="controller_plugins" params="namespace">
+        <ros2_control name="GazeboSystem" type="system">
+            <hardware>
+                <plugin>gazebo_ros2_control/GazeboSystem</plugin>
+            </hardware>
+            <xacro:macro name="robot_joint" params="link_id">
+                <joint name="joint_${link_id}">
+                    <command_interface name="position">
+                        <param name="min">-3.14</param>
+                        <param name="max">3.14</param>
+                    </command_interface>
+                    <state_interface name="position">
+                        <param name="initial_value">0.0</param>
+                    </state_interface>
+                    <state_interface name="velocity"/>
+                    <state_interface name="effort"/>
+                </joint>
+            </xacro:macro>
+            <xacro:robot_joint link_id="1"/>
+            <xacro:robot_joint link_id="2"/>
+            <xacro:robot_joint link_id="3"/>
+        </ros2_control>
+        <gazebo>
+            <plugin filename="libgazebo_ros2_control.so" name="gazebo_ros2_joint_control">
+                <parameters>$(find dummy_gazebo)/config/${namespace}_controller_config.yaml</parameters>
+                <ros>
+                    <namespace>/${namespace}</namespace>
+                </ros>
+            </plugin>
+        </gazebo>
+    </xacro:macro>
 </robot>
