Commit message: Add files via upload

File: mobile_robot/xxx_gazebo/robot/ros2_control.gazebo.xacro (robot description, xacro)
@@ -1,3 +1,28 @@
 <?xml version='1.0' encoding='utf-8'?>
-<robot xmlns:xacro="http://www.ros.org/wiki/xacro" name="xxx">
+<robot xmlns:xacro="http://www.ros.org/wiki/xacro">
+    <xacro:macro name="controller_plugins" params="namespace">
+        <ros2_control name="GazeboSystem" type="system">
+            <hardware>
+                <plugin>gazebo_ros2_control/GazeboSystem</plugin>
+            </hardware>
+            <xacro:macro name="wheel_joint" params="joint_name">
+                <joint name="${joint_name}">
+                    <command_interface name="velocity"/>
+                    <command_interface name="effort"/>
+                    <state_interface name="velocity"/>
+                    <state_interface name="effort"/>
+                </joint>
+            </xacro:macro>
+            <xacro:wheel_joint joint_name="left_wheel_joint"/>
+            <xacro:wheel_joint joint_name="right_wheel_joint"/>
+        </ros2_control>
+        <gazebo>
+            <plugin filename="libgazebo_ros2_control.so" name="gazebo_ros2_wheel_control">
+                <parameters>$(find xxx_gazebo)/config/${namespace}_controller_config.yaml</parameters>
+                <ros>
+                    <namespace>/${namespace}</namespace>
+                </ros>
+            </plugin>
+        </gazebo>
+    </xacro:macro>
 </robot>

File: mobile_robot/xxx_gazebo/robot/xxx.xacro (robot description, xacro)
@@ -1,4 +1,6 @@
 <?xml version='1.0' encoding='utf-8'?>
 <robot xmlns:xacro="http://www.ros.org/wiki/xacro" name="xxx">
+  <xacro:arg name="robot_name" default=""/>
+  <xacro:property name="namespace" value="$(arg robot_name)"/>
   <xacro:include filename="$(find xxx_description)/robot/dynamics/physical_robot.xacro"/>
   <xacro:include filename="$(find xxx_gazebo)/robot/graphics.gazebo.xacro"/>
@@ -7,3 +9,4 @@
   <xacro:physical_robot/>
   <xacro:gazebo_graphics/>
+  <xacro:controller_plugins namespace="${namespace}"/>
 </robot>
